Commit message: added caster

File: diff_drive/urdf/robot.urdf.xacro (robot description, xacro)
@@ -3,11 +3,59 @@
     <xacro:property name="yaml_file" value="$(find diff_drive)/config/robot_size.yaml" />
     <xacro:property name="props" value="${xacro.load_yaml(yaml_file)['/**']['ros__parameters']}" />
-    <xacro:include filename="$(find diff_drive)/urdf/_base_link.urdf.xacro" />
-    <xacro:base_link name="base_link"/>
-    <link name="base_footprint"/>
-    <joint name="base_link_to_base_footprint" type="fixed">
-        <origin xyz="0 0 -0.5" rpy="0 0 0"/>
+    <xacro:property name="base_link_length"  value="${props['base_link_length']}" />
+    <xacro:property name="base_link_width"  value="${props['base_link_width']}" />
+    <xacro:property name="base_link_height"  value="${props['base_link_height']}" />
+    <xacro:property name="wheel_radius"  value="${props['wheel_radius']}" />
+    <xacro:property name="wheel_height"  value="${props['wheel_height']}" />
+    <xacro:property name="PI"  value="3.1415926535897932" />
+    <xacro:include filename="$(find diff_drive)/urdf/_wheel.urdf.xacro" />
+    <xacro:include filename="$(find diff_drive)/urdf/_caster.urdf.xacro" />
+    <link name="base_link">
+        <visual>
+            <geometry>
+                <box size="${base_link_length} ${base_link_width} ${base_link_height}"/>
+            </geometry>
+            <material name="base_link_color">
+                <color rgba="0.0 0.0 1.0 1.0"/>
+            </material>
+        </visual>
+    </link>
+    <xacro:wheel name="left_wheel"/>
+    <xacro:wheel name="right_wheel"/>
+    <xacro:caster name="up_caster"/>
+    <xacro:caster name="bottom_caster"/>
+    <joint name="base_link_to_left_wheel" type="continuous">
         <parent link="base_link"/>
-        <child link="base_footprint"/>
+        <child link="left_wheel"/>
+        <axis xyz="0 1 0"/>
+        <origin xyz="${base_link_length/2 - base_link_height/2}
+                     ${base_link_width/2 + wheel_height/2}
+                     0" rpy="0 0 0"/>
+        <limit effort="10.0" velocity="10.0"/>
+    </joint>
+    <joint name="base_link_to_right_wheel" type="continuous">
+        <parent link="base_link"/>
+        <child link="right_wheel"/>
+        <axis xyz="0 1 0"/>
+        <origin xyz="${base_link_length/2 - base_link_height/2}
+                     ${-base_link_width/2 - wheel_height/2}
+                     0" rpy="0 0 0"/>
+        <limit effort="10.0" velocity="10.0"/>
+    </joint>
+    <joint name="base_link_to_up_caster" type="fixed">
+        <parent link="base_link"/>
+        <child link="up_caster"/>
+        <origin xyz="-${base_link_length/2 - wheel_radius + base_link_height/2}
+                     0
+                     ${base_link_height/2}" rpy="0 0 0"/>
+        <limit effort="10.0" velocity="10.0"/>
+    </joint>
+    <joint name="base_link_to_bottom_caster" type="fixed">
+        <parent link="base_link"/>
+        <child link="bottom_caster"/>
+        <origin xyz="-${base_link_length/2 - wheel_radius + base_link_height/2}
+                     0
+                     ${-base_link_height/2}" rpy="0 0 0"/>
+        <limit effort="10.0" velocity="10.0"/>
     </joint>
 </robot>
