Commit message: spawned urdf

File: diff_drive/urdf/_caster.urdf.xacro (robot description, xacro)
@@ -7,7 +7,15 @@
     <xacro:property name="wheel_radius"  value="${props['wheel_radius']}" />
     <xacro:property name="wheel_height"  value="${props['wheel_height']}" />
+    <xacro:property name="caster_mass"  value="${props['caster_mass']}" />
     <xacro:property name="PI"  value="3.1415926535897932" />
     <xacro:macro name="caster" params="name">
         <link name="${name}">
+            <inertial>
+                <origin xyz="0 0 0" rpy="0 0 0"/>
+                <mass value="${caster_mass}"/>
+                <inertia ixx="${caster_mass * (2/5) * (wheel_radius**2)}" ixy="0" ixz="0"
+                         iyx="0" iyy="${caster_mass * (2/5) * (wheel_radius**2)}" iyz="0"
+                         izx="0" izy="0" izz="${caster_mass * (2/5) * (wheel_radius**2)}"/>
+            </inertial>
             <visual>
                 <origin xyz="0 0 0" rpy="${PI/2} 0 0"/>

File: diff_drive/urdf/_wheel.urdf.xacro (robot description, xacro)
@@ -4,7 +4,15 @@
     <xacro:property name="wheel_radius"  value="${props['wheel_radius']}" />
     <xacro:property name="wheel_height"  value="${props['wheel_height']}" />
+    <xacro:property name="wheel_mass"  value="${props['wheel_mass']}" />
     <xacro:property name="PI"  value="3.1415926535897932" />
     <xacro:macro name="wheel" params="name">
         <link name="${name}">
+            <inertial>
+                <origin xyz="0 0 0" rpy="0 0 0"/>
+                <mass value="${wheel_mass}"/>
+                <inertia ixx="${wheel_mass * (2/5) * (wheel_radius**2)}" ixy="0" ixz="0"
+                         iyx="0" iyy="${wheel_mass * (2/5) * (wheel_radius**2)}" iyz="0"
+                         izx="0" izy="0" izz="${wheel_mass * (2/5) * (wheel_radius**2)}"/>
+            </inertial>
             <visual>
                 <origin xyz="0 0 0" rpy="${PI/2} 0 0"/>

File: diff_drive/urdf/ddrive.gazebo.xacro (robot description, xacro)
@@ -6,4 +6,5 @@
     <xacro:property name="base_link_width"  value="${props['base_link_width']}" />
     <xacro:property name="base_link_height"  value="${props['base_link_height']}" />
+    <xacro:property name="base_link_mass"  value="${props['base_link_mass']}" />
     <xacro:property name="wheel_radius"  value="${props['wheel_radius']}" />
     <xacro:property name="wheel_height"  value="${props['wheel_height']}" />
@@ -12,4 +13,11 @@
     <xacro:include filename="$(find diff_drive)/urdf/_caster.urdf.xacro" />
     <link name="base_link">
+        <inertial>
+            <origin xyz="0 0 0" rpy="0 0 0"/>
+            <mass value="${base_link_mass}"/>
+            <inertia ixx="${base_link_mass * (base_link_width**2 + base_link_height**2) / 12}" ixy="0" ixz="0"
+                     iyx="0" iyy="${base_link_mass * (base_link_length**2 + base_link_height**2) / 12}" iyz="0"
+                     izx="0" izy="0" izz="${base_link_mass * (base_link_length**2 + base_link_width**2) / 12}"/>
+        </inertial>
         <visual>
             <geometry>
@@ -20,4 +28,9 @@
             </material>
         </visual>
+        <collision>
+            <geometry>
+                <box size="${base_link_length} ${base_link_width} ${base_link_height}"/>
+            </geometry>
+        </collision>
     </link>
     <xacro:wheel name="left_wheel"/>
@@ -59,3 +72,25 @@
         <limit effort="10.0" velocity="10.0"/>
     </joint>
+    <gazebo>
+        <plugin name="gz::sim::systems::DiffDrive" filename="gz-sim-diff-drive-system">
+        <rosDebugLevel>na</rosDebugLevel>
+        <alwaysOn>true</alwaysOn>
+        <updateRate>100</updateRate>
+        <leftJoint>base_link_to_left_wheel</leftJoint>
+        <rightJoint>base_link_to_right_wheel</rightJoint>
+        <wheelSeparation>${base_link_width+wheel_height}</wheelSeparation>
+        <wheelDiameter>${wheel_radius*2}</wheelDiameter>
+        <wheelTorque>20</wheelTorque>
+        <commandTopic>cmd_vel</commandTopic>
+        <odometryTopic>odom</odometryTopic>
+        <odometryFrame>odom</odometryFrame>
+        <robotBaseFrame>base_link</robotBaseFrame>
+        <publishWheelTF>false</publishWheelTF>
+        <publishOdomTF>true</publishOdomTF>
+        <publishWheelJointState>true</publishWheelJointState>
+        <wheelAcceleration>false</wheelAcceleration>
+        <odometrySource>world</odometrySource>
+        <publishTf>1</publishTf>
+        </plugin>
+    </gazebo>
 </robot>
